File: dod-juice-box-clone.kicad_pcb (KiCad board)
At the start: 2 copper layers, 55 x 46 mm, 64 parts, among them Q1 J201, Q2 2N5088, Q3 2N5088, Q4 2N5088, U1 RC4558

Commit message: Stopping point
Parts:
- moved C10 13.9 mm to (91.6, 43.0)
- moved C17 13.9 mm to (101.3, 52.0)
- moved C1 13.9 mm to (91.6, 18.6)
- moved C11 13.9 mm to (91.6, 47.0)
- moved C12 13.9 mm to (91.6, 51.0)
- moved C13 13.9 mm to (91.6, 55.1)
- moved C14 13.9 mm to (101.3, 36.2)
- moved C15 13.9 mm to (91.6, 59.1)
- moved C16 13.9 mm to (101.3, 44.1)
- moved C2 13.9 mm to (91.6, 22.7)
- moved C4 13.9 mm to (91.6, 26.8)
- moved C5 13.9 mm to (91.6, 30.8)
- moved C6 13.9 mm to (91.6, 34.9)
- moved C7 13.9 mm to (91.6, 38.9)
- moved C8 13.9 mm to (101.3, 20.6)
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Other:
- board size 55 x 46 mm -> 53 x 64.5 mm
- board text added: "Update PCB with new pot footprint and finish layout"
- board text removed: "TODO: measure PCB size if I put LED on right of switch instead of top"
